Commit message: change urdf
small change in urdf

File: 1_Mechanic/alexbotmini_urdf/alexbotmini/urdf/alexbotmini.urdf (robot description, URDF)
Before this commit: robot alexbotmini, 13 links, 12 joints
Links:
- link base_link: mass 7.3572 -> 7.35718055319755
- link leftlink1: mass 0.52383 -> 0.523827453897711
- link leftlink2: mass 0.95964 -> 0.959639548121109
- link leftlink3: mass 0.81627 -> 0.816268978197084
- link leftlink4: mass 1.192 -> 1.19197432366853
- link leftlink5: mass 0.017311 -> 0.0173110583311115
- link leftlink6: mass 0.62406 -> 0.624059283851391
- link rightlink1: mass 0.52383 -> 0.523827457014568
- link rightlink3: mass 0.81499 -> 0.81499254145314
- link rightlink5: mass 0.0173110583311114 -> 0.0173110583311115
Joints:
- joint leftjoint3: axis 0 1 0 -> 0 0 1
- joint leftjoint4: axis 0 0 1 -> 1 0 0
- joint leftjoint5: origin xyz=0.021108 0.0032246 -0.28934 rpy=0 0 0 -> xyz=0.021337 -0.0042697 -0.28916 rpy=0 0 0
- joint rightjoint2: axis 0 -1 0 -> 0 1 0; origin xyz=0.052 -0.081589 0.0013677 rpy=0 0 0 -> xyz=0.052 -0.081599 -0.00047085 rpy=0 0 0
- joint rightjoint3: axis 0 0 -1 -> 0 0 1; origin xyz=-0.0027097 0.07579 -0.15965 rpy=0 0 0 -> xyz=0.001813 0.079368 -0.15792 rpy=0 0 0
- joint rightjoint4: origin xyz=0.024553 -0.0029335 -0.14241 rpy=0 0 0 -> xyz=0.028485 -0.0014832 -0.1417 rpy=0 0 0
- joint rightjoint5: origin xyz=-0.029608 0.0055383 -0.28845 rpy=0 0 0 -> xyz=-0.02312 -0.010345 -0.28903 rpy=0 0 0
- joint rightjoint6: axis 1 0 0 -> -1 0 0
